File: kicad/adapter_soic8_solder/adapter_soic8_solder.kicad_pcb (KiCad board)
At the start: 2 copper layers, 48 x 20 mm, 3 parts, among them J1 Conn_02x07_Odd_Even, J2 Conn_02x07_Odd_Even, U1 AT45DB

Commit message: Revert "upgrade project files to kicad version 6.0.11"
This reverts commit 6c6c989fefeeef77173a4749b3826cd3583d0fba.
Other:
- net class Default added: clearance 0.2, trace_width 0.25, via_dia 0.8, via_drill 0.4

Commit message: upgrade project files to kicad version 6.0.11
Other:
- net class Default removed
